File: SoftKeyboardController/temp.kicad_sch (KiCad schematic)
At the start: 40 parts, among them IC1 PCA9956BTWY, J1 Barrel_Jack, J2 Conn_01x08_Socket, J3 Motor 1, J4 Motor 2, J5 Conn_01x12_Socket, J6 Conn_01x12_Socket, J7 EXT IMU Connection, J8 Conn_01x08_Socket, Q1 Q_NMOS_GDS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

Commit message: Added Transistors & ADCs to schematic. V1 of PCB
Parts:
- added H1, H2, H3, H4: MountingHole, MountingHole:MountingHole_2.5mm, symbol Mechanical:MountingHole
Connections:
- net +3V3: no longer J7.4 (Pin_4)
- net GND: no longer J1.2, J7.5 (Pin_5)
- net SCL: no longer J7.2 (Pin_2)
- net SDA: no longer J7.1 (Pin_1)
- net at C1.1, C2.2, U1.12 (VM): no longer J1.1
- net at ESP1.35 (GPIO1/TX0), IC1.35 (~{RESET}), R5.2: no longer J7.3 (Pin_3)
Other:
- moved on the sheet: C1, C2, C4, C5, ESP1, IC1, J2, J3, J4, J5, J6, J8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
