File: hardware/SoftKeyboardController.kicad_pcb (KiCad board)
At the start: 2 copper layers, 87.1 x 78.7 mm, 52 parts, among them IC1 PCA9956BTWY, J1 Barrel_Jack_Switch, J10 Motor Encoder 1, J2 EXT IMU Connection, J3 Motor 1, J4 Motor 2, J5 Conn_01x12_Socket, J6 Conn_01x12_Socket, J7 Conn_01x08_Socket, J8 Conn_01x08_Socket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

Commit message: rename hardware folder for clarity
Parts:
- R10, R11, R8, R9: value 470Ω -> 1kΩ
Changed lines of the file:
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@@
 		(tags "Integrated Circuit")
 		(property "Reference" "IC1"
-			(at -0.0726 -6.0152 90)
+			(at -0.038939 -6.232097 90)
 			(layer "F.SilkS")
 			(effects
@@
 			)
 		)
-		(property "Value" "470Ω"
+		(property "Value" "1kΩ"
 			(at 0 2.921 90)
 			(layer "F.SilkS")
@@
 			)
 		)
-		(property "Value" "470Ω"
+		(property "Value" "1kΩ"
 			(at 0 2.794 90)
 			(layer "F.SilkS")
@@
 		(tags "test point wire loop bead")
 		(property "Reference" "TP11"
-			(at 0.103521 2.562239 0)
+			(at -0.216846 2.30508 0)
 			(layer "F.SilkS")
 			(effects
@@
 			)
 		)
-		(property "Value" "470Ω"
+		(property "Value" "1kΩ"
 			(at -0.1505 3.048 90)
 			(layer "F.SilkS")
@@
 			)
 		)
-		(property "Value" "470Ω"
+		(property "Value" "1kΩ"
 			(at 0 2.921 90)
 			(layer "F.SilkS")
@@
 	)
 	(via
-		(at 172.466 100.637)
+		(at 172.520718 100.815626)
 		(size 0.6)
 		(drill 0.3)
@@
 	)
 	(via
-		(at 171.196 101.272)
+		(at 171.250718 101.450626)
 		(size 0.6)
 		(drill 0.3)
@@
 	)
 	(via
-		(at 172.466 101.907)
+		(at 172.520718 102.085626)
 		(size 0.6)
 		(drill 0.3)
@@
 	)
 	(via
-		(at 171.196 100.002)
+		(at 171.250718 100.180626)
 		(size 0.6)
 		(drill 0.3)
@@
 	)
 	(via
-		(at 171.196 100.637)
+		(at 171.250718 100.815626)
 		(size 0.6)
 		(drill 0.3)
@@
 	)
 	(via
-		(at 171.831 100.637)
+		(at 171.885718 100.815626)
 		(size 0.6)
 		(drill 0.3)
@@
 	)
 	(via
-		(at 171.831 101.907)
+		(at 171.885718 102.085626)
 		(size 0.6)
 		(drill 0.3)
@@
 	)
 	(via
-		(at 172.466 101.272)
+		(at 172.520718 101.450626)
 		(size 0.6)
 		(drill 0.3)
@@
 	)
 	(via
-		(at 171.196 101.907)
+		(at 171.250718 102.085626)
 		(size 0.6)
 		(drill 0.3)
@@
 	)
 	(via
-		(at 171.831 101.272)
+		(at 171.885718 101.450626)
 		(size 0.6)
 		(drill 0.3)
@@
 	)
 	(via
-		(at 171.831 100.002)
+		(at 171.885718 100.180626)
 		(size 0.6)
 		(drill 0.3)
@@
 	)
 	(via
-		(at 172.466 100.002)
+		(at 172.520718 100.180626)
 		(size 0.6)
 		(drill 0.3)

Commit message: small change to board reflecting fixed SCL and SDA miswiring
Parts:
- moved R6 9.65 mm to (225.8, 93.3)
- moved R2 9.61 mm to (216.2, 93.3)
Connections:
- ESP1 pad 33: SCL -> SDA
- ESP1 pad 36: SDA -> SCL
- IC1 pad 5: unconnected-(IC1-~{OE}-Pad5) -> GND
- R2 pad 2: SDA -> SCL
- R6 pad 2: SCL -> SDA
- TP3 pad 1: SDA -> SCL
- TP4 pad 1: SCL -> SDA
Routing:
- net SCL: track 152.4 -> 159.8 mm, vias 8 -> 10
- net GND: track 77.6 -> 80.3 mm
- net SDA: track 158.6 -> 159.3 mm, vias 8 -> 10
