File: hardware/SoftKeyboardController.kicad_sch (KiCad schematic)
At the start: 52 parts, among them IC1 PCA9956BTWY, J1 Barrel_Jack_Switch, J10 Motor Encoder 1, J2 EXT IMU Connection, J3 Motor 1, J4 Motor 2, J5 Conn_01x12_Socket, J6 Conn_01x12_Socket, J7 Conn_01x08_Socket, J8 Conn_01x08_Socket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

Commit message: rename hardware folder for clarity
Parts:
- R10, R11, R8, R9: value 470Ω -> 1kΩ
Changed lines of the file:
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@@
 			)
 		)
-		(property "Value" "470Ω"
+		(property "Value" "1kΩ"
 			(at 183.896 199.898 90)
 			(effects
@@
 			)
 		)
-		(property "Value" "470Ω"
+		(property "Value" "1kΩ"
 			(at 184.404 180.848 90)
 			(effects
@@
 			)
 		)
-		(property "Value" "470Ω"
+		(property "Value" "1kΩ"
 			(at 184.404 191.77 90)
 			(effects
@@
 					(size 1.27 1.27)
 				)
-				(hide yes)
 			)
 		)
@@
 			)
 		)
-		(property "Value" "470Ω"
+		(property "Value" "1kΩ"
 			(at 184.404 211.328 90)
 			(effects

Commit message: small change to board reflecting fixed SCL and SDA miswiring
Connections:
- net GND: now also IC1.5 (~{OE})
- net SCL: now also ESP1.36 (GPIO22/SCL), R2.2, TP3.1; no longer ESP1.33 (GPIO21/SDA), R6.2, TP4.1
- net SDA: now also ESP1.33 (GPIO21/SDA), R6.2, TP4.1; no longer ESP1.36 (GPIO22/SCL), R2.2, TP3.1
Changed lines of the file:
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@@
 	)
 	(junction
+		(at 326.39 57.15)
+		(diameter 0)
+		(color 0 0 0 0)
+	)
+	(junction
 		(at 143.51 142.24)
 		(diameter 0)
@@
 	(wire
 		(pts
+			(xy 325.12 59.69) (xy 326.39 59.69)
+		)
+		(stroke
+			(width 0)
+			(type default)
+		)
+	)
+	(wire
+		(pts
+			(xy 326.39 59.69) (xy 326.39 57.15)
+		)
+		(stroke
+			(width 0)
+			(type default)
+		)
+	)
+	(wire
+		(pts
 			(xy 287.02 127) (xy 287.02 128.27)
 		)
@@
 	(global_label "SDA"
 		(shape input)
-		(at 223.52 111.76 0)
+		(at 233.68 114.3 0)
 		(fields_autoplaced yes)
 		(effects
@@
 		)
 		(property "Intersheetrefs" "${INTERSHEET_REFS}"
-			(at 230.0733 111.76 0)
+			(at 240.2333 114.3 0)
 			(effects
 				(font
@@
 		)
 	)
-	(global_label "s2"
+	(global_label "SCL"
 		(shape input)
-		(at 77.47 111.76 180)
+		(at 223.52 111.76 0)
 		(fields_autoplaced yes)
 		(effects
@@
 				(size 1.27 1.27)
 			)
-			(justify right)
+			(justify left)
 		)
 		(property "Intersheetrefs" "${INTERSHEET_REFS}"
-			(at 72.2472 111.76 0)
+			(at 230.0128 111.76 0)
 			(effects
 				(font
 					(size 1.27 1.27)
 				)
-				(justify right)
+				(justify left)
 				(hide yes)
 			)
 		)
 	)
-	(global_label "5v"
+	(global_label "s2"
 		(shape input)
-		(at 199.39 104.14 90)
+		(at 77.47 111.76 180)
 		(fields_autoplaced yes)
 		(effects
@@
 				(size 1.27 1.27)
 			)
-			(justify left)
+			(justify right)
 		)
 		(property "Intersheetrefs" "${INTERSHEET_REFS}"
-			(at 199.39 98.9777 90)
+			(at 72.2472 111.76 0)
 			(effects
 				(font
 					(size 1.27 1.27)
 				)
-				(justify left)
+				(justify right)
 				(hide yes)
 			)
 		)
 	)
-	(global_label "I_Op"
+	(global_label "5v"
 		(shape input)
-		(at 177.8 119.38 180)
+		(at 199.39 104.14 90)
 		(fields_autoplaced yes)
 		(effects
@@
 				(size 1.27 1.27)
 			)
-			(justify right)
+			(justify left)
 		)
 		(property "Intersheetrefs" "${INTERSHEET_REFS}"
-			(at 170.7629 119.38 0)
+			(at 199.39 98.9777 90)
 			(effects
 				(font
 					(size 1.27 1.27)
 				)
-				(justify right)
+				(justify left)
 				(hide yes)
 			)
 		)
 	)
-	(global_label "SCL"
+	(global_label "I_Op"
 		(shape input)
-		(at 233.68 114.3 0)
+		(at 177.8 119.38 180)
 		(fields_autoplaced yes)
 		(effects
@@
 				(size 1.27 1.27)
 			)
-			(justify left)
+			(justify right)
 		)
 		(property "Intersheetrefs" "${INTERSHEET_REFS}"
-			(at 240.1728 114.3 0)
+			(at 170.7629 119.38 0)
 			(effects
 				(font
 					(size 1.27 1.27)
 				)
-				(justify left)
+				(justify right)
 				(hide yes)
 			)
